File: board/OmniView.brd (EAGLE design)
At the start: 160 x 100 mm, 50 parts, among them Q1 CMA-4544PF-W, Q2 BSS138, Q3 BSS138, U1 SN74LVC2T45DCUT, U2 UG-2864HSWEG01

Commit message: schematic check-up
did a little bit of schematic setting up
Parts:
- added 32KHZ: ABS07, ABS07_crys:ABS07
- added C14, C15: 10pF, rcl:C0603
- added C16: 10uF, rcl:C0603
- added C17, C18, C19, C20: .1uF, rcl:C0603
- added C21, C22, C23: 4.7uF, rcl:C0603
- added U$27: 2.2uH, ABS07_crys:1008INDUCTOR
- added U$4: Q24FA20H00396, ABS07_crys:Q24FA20H00396
Connections:
- removed net DCDC_DIG_SW: CC1.43
- removed net GND_TAB: CC1.65
- removed net VCC: IC1.3, IC1.42
- removed net VDD_DIG1: CC1.9
- removed net VDD_DIG2: CC1.56
- removed net VIN_DCDC_ANA: CC1.37
- removed net VIN_DCDC_DIG: CC1.44
- removed net VIN_DCDC_PA: CC1.39
- removed net VIN_IO1: CC1.10
- removed net VIN_IO2: CC1.54
- new net N$18: CC1.43, U$27.P2
- new net N$19: C16.1, U$27.P1
- new net N$20: C17.1, C18.1, CC1.56, CC1.9
- new net VBAT_CC: C19.1, C20.1, C21.1, C22.1, C23.1, CC1.10, CC1.37, CC1.39, CC1.44, CC1.54, IC1.3, IC1.42
- new net XHIGH: CC1.23, U$4.XHIGH
- new net XLOW: CC1.22, U$4.XLOW
- new net XTALHIGH: 32KHZ.XLOW, C15.1, CC1.51
- new net XTALLOW: 32KHZ.XHIGH, C14.2, CC1.52
- net GND: now also C14.1, C15.2, C16.2, C17.2, C18.2, C19.2, C20.2, C21.2, C22.2, C23.2, CC1.65, U$4.GND1, U$4.GND2
Changed lines of the file:
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@@
 <element name="U$26" library="microbuilder" package="MOUNTINGHOLE_2.5_PLATED" value="MOUNTINGHOLE2.5" x="23" y="-79"/>
 <element name="IC1" library="ftdichip-3" package="QFP48-7X7" value="" x="8" y="-105"/>
+<element name="C14" library="rcl" package="C0603" value="10pF" x="2" y="-113"/>
+<element name="C15" library="rcl" package="C0603" value="10pF" x="2" y="-117"/>
+<element name="32KHZ" library="ABS07_crys" package="ABS07" value="ABS07" x="3" y="-121"/>
+<element name="U$4" library="ABS07_crys" package="Q24FA20H00396" value="Q24FA20H00396" x="2" y="-124"/>
+<element name="C19" library="rcl" package="C0603" value=".1uF" x="2" y="-141"/>
+<element name="C20" library="rcl" package="C0603" value=".1uF" x="2" y="-145"/>
+<element name="C21" library="rcl" package="C0603" value="4.7uF" x="2" y="-150"/>
+<element name="C22" library="rcl" package="C0603" value="4.7uF" x="2" y="-154"/>
+<element name="C23" library="rcl" package="C0603" value="4.7uF" x="2" y="-158"/>
+<element name="U$27" library="ABS07_crys" package="1008INDUCTOR" value="2.2uH" x="2" y="-162"/>
+<element name="C16" library="rcl" package="C0603" value="10uF" x="2" y="-166"/>
+<element name="C17" library="rcl" package="C0603" value=".1uF" x="2" y="-171"/>
+<element name="C18" library="rcl" package="C0603" value=".1uF" x="2" y="-176"/>
 </elements>
 <signals>
-<signal name="VDD_DIG1">
-<contactref element="CC1" pad="9"/>
-</signal>
-<signal name="VIN_IO1">
-<contactref element="CC1" pad="10"/>
-</signal>
 <signal name="VDD_PLL">
 <contactref element="CC1" pad="24"/>
@@
 <contactref element="CC1" pad="36"/>
 </signal>
-<signal name="VIN_DCDC_ANA">
-<contactref element="CC1" pad="37"/>
-</signal>
 <signal name="DCDC_ANA_SW">
 <contactref element="CC1" pad="38"/>
 </signal>
-<signal name="VIN_DCDC_PA">
-<contactref element="CC1" pad="39"/>
-</signal>
 <signal name="DCDC_PA_SW_P">
 <contactref element="CC1" pad="40"/>
@@
 <contactref element="CC1" pad="42"/>
 </signal>
-<signal name="DCDC_DIG_SW">
-<contactref element="CC1" pad="43"/>
-</signal>
-<signal name="VIN_DCDC_DIG">
-<contactref element="CC1" pad="44"/>
-</signal>
 <signal name="VDD_ANA2">
 <contactref element="CC1" pad="47"/>
@@
 <signal name="VDD_RAM">
 <contactref element="CC1" pad="49"/>
-</signal>
-<signal name="VIN_IO2">
-<contactref element="CC1" pad="54"/>
-</signal>
-<signal name="VDD_DIG2">
-<contactref element="CC1" pad="56"/>
-</signal>
-<signal name="GND_TAB">
-<contactref element="CC1" pad="65"/>
 </signal>
 <signal name="VCCA">
@@
 <contactref element="IC1" pad="18"/>
 <contactref element="IC1" pad="9"/>
+<contactref element="C14" pad="1"/>
+<contactref element="C15" pad="2"/>
+<contactref element="U$4" pad="GND1"/>
+<contactref element="U$4" pad="GND2"/>
+<contactref element="CC1" pad="65"/>
+<contactref element="C23" pad="2"/>
+<contactref element="C21" pad="2"/>
+<contactref element="C22" pad="2"/>
+<contactref element="C19" pad="2"/>
+<contactref element="C20" pad="2"/>
+<contactref element="C16" pad="2"/>
+<contactref element="C17" pad="2"/>
+<contactref element="C18" pad="2"/>
+<wire x1="2.85" y1="-171" x2="2.85" y2="-176" width="0" layer="19" extent="1-1"/>
+<wire x1="2.85" y1="-166" x2="2.85" y2="-171" width="0" layer="19" extent="1-1"/>
+<wire x1="2.85" y1="-158" x2="2.85" y2="-166" width="0" layer="19" extent="1-1"/>
+<wire x1="2.85" y1="-154" x2="2.85" y2="-158" width="0" layer="19" extent="1-1"/>
+<wire x1="2.85" y1="-150" x2="2.85" y2="-154" width="0" layer="19" extent="1-1"/>
+<wire x1="2.85" y1="-145" x2="2.85" y2="-150" width="0" layer="19" extent="1-1"/>
+<wire x1="2.85" y1="-141" x2="2.85" y2="-145" width="0" layer="19" extent="1-1"/>
+<wire x1="2.8636" y1="-124.6858" x2="2.85" y2="-141" width="0" layer="19" extent="1-1"/>
+<wire x1="1.1618" y1="-123.2888" x2="2.8636" y2="-124.6858" width="0" layer="19" extent="1-1"/>
+<wire x1="2.85" y1="-117" x2="1.1618" y2="-123.2888" width="0" layer="19" extent="1-1"/>
+<wire x1="1.15" y1="-113" x2="2.85" y2="-117" width="0" layer="19" extent="1-1"/>
+<wire x1="9.25" y1="-109.15" x2="1.15" y2="-113" width="0" layer="19" extent="1-1"/>
 <wire x1="12.15" y1="-105.25" x2="9.25" y2="-109.15" width="0" layer="19" extent="1-1"/>
 <wire x1="10.75" y1="-100.85" x2="12.15" y2="-105.25" width="0" layer="19" extent="1-1"/>
@@
 <wire x1="21.475" y1="-20" x2="20" y2="-20" width="0" layer="19" extent="1-1"/>
 <wire x1="10.7" y1="-20" x2="18.525" y2="-20" width="0" layer="19" extent="1-1"/>
+<wire x1="57.015" y1="42.3694" x2="21.475" y2="-20" width="0" layer="19" extent="1-1"/>
 </signal>
 <signal name="INPUT">
@@
 <contactref element="IC1" pad="46"/>
 </signal>
-<signal name="VCC">
+<signal name="VBAT_CC">
 <contactref element="IC1" pad="3"/>
 <contactref element="IC1" pad="42"/>
+<contactref element="C21" pad="1"/>
+<contactref element="C23" pad="1"/>
+<contactref element="C22" pad="1"/>
+<contactref element="C19" pad="1"/>
+<contactref element="C20" pad="1"/>
+<contactref element="CC1" pad="10"/>
+<contactref element="CC1" pad="54"/>
+<contactref element="CC1" pad="44"/>
+<contactref element="CC1" pad="39"/>
+<contactref element="CC1" pad="37"/>
+<wire x1="1.15" y1="-154" x2="1.15" y2="-158" width="0" layer="19" extent="1-1"/>
+<wire x1="1.15" y1="-150" x2="1.15" y2="-154" width="0" layer="19" extent="1-1"/>
+<wire x1="1.15" y1="-145" x2="1.15" y2="-150" width="0" layer="19" extent="1-1"/>
+<wire x1="1.15" y1="-141" x2="1.15" y2="-145" width="0" layer="19" extent="1-1"/>
+<wire x1="6.25" y1="-109.15" x2="1.15" y2="-141" width="0" layer="19" extent="1-1"/>
 <wire x1="3.85" y1="-104.75" x2="6.25" y2="-109.15" width="0" layer="19" extent="1-1"/>
+<wire x1="55.265" y1="37.8694" x2="3.85" y2="-104.75" width="0" layer="19" extent="1-1"/>
+<wire x1="56.265" y1="37.8694" x2="55.265" y2="37.8694" width="0" layer="19" extent="1-1"/>
+<wire x1="58.765" y1="37.8694" x2="56.265" y2="37.8694" width="0" layer="19" extent="1-1"/>
+<wire x1="61.515" y1="41.1194" x2="58.765" y2="37.8694" width="0" layer="19" extent="1-1"/>
+<wire x1="56.265" y1="46.8694" x2="61.515" y2="41.1194" width="0" layer="19" extent="1-1"/>
 </signal>
 <signal name="3V3OUT">
@@
 <contactref element="IC1" pad="14"/>
 </signal>
+<signal name="XTALLOW">
+<contactref element="C14" pad="2"/>
+<contactref element="CC1" pad="52"/>
+<contactref element="32KHZ" pad="XHIGH"/>
+<wire x1="2.85" y1="-113" x2="1.73" y2="-121" width="0" layer="19" extent="1-1"/>
+<wire x1="61.515" y1="40.1194" x2="2.85" y2="-113" width="0" layer="19" extent="1-1"/>
+</signal>
+<signal name="XTALHIGH">
+<contactref element="CC1" pad="51"/>
+<contactref element="32KHZ" pad="XLOW"/>
+<contactref element="C15" pad="1"/>
+<wire x1="1.15" y1="-117" x2="4.27" y2="-121" width="0" layer="19" extent="1-1"/>
+<wire x1="61.515" y1="39.6194" x2="1.15" y2="-117" width="0" layer="19" extent="1-1"/>
+</signal>
+<signal name="XHIGH">
+<contactref element="U$4" pad="XHIGH"/>
+<contactref element="CC1" pad="23"/>
+<wire x1="52.515" y1="43.1194" x2="2.8636" y2="-123.2888" width="0" layer="19" extent="1-1"/>
+</signal>
+<signal name="XLOW">
+<contactref element="U$4" pad="XLOW"/>
+<contactref element="CC1" pad="22"/>
+<wire x1="52.515" y1="43.6194" x2="1.1618" y2="-124.6858" width="0" layer="19" extent="1-1"/>
+</signal>
+<signal name="N$18">
+<contactref element="CC1" pad="43"/>
+<contactref element="U$27" pad="P2"/>
+<wire x1="58.265" y1="37.8694" x2="3.25" y2="-161.95" width="0" layer="19" extent="1-1"/>
+</signal>
+<signal name="N$19">
+<contactref element="U$27" pad="P1"/>
+<contactref element="C16" pad="1"/>
+<wire x1="0.7" y1="-161.975" x2="1.15" y2="-166" width="0" layer="19" extent="1-1"/>
+</signal>
+<signal name="N$20">
+<contactref element="CC1" pad="9"/>
+<contactref element="CC1" pad="56"/>
+<contactref element="C17" pad="1"/>
+<contactref element="C18" pad="1"/>
+<wire x1="1.15" y1="-171" x2="1.15" y2="-176" width="0" layer="19" extent="1-1"/>
+<wire x1="61.515" y1="42.1194" x2="1.15" y2="-171" width="0" layer="19" extent="1-1"/>
+<wire x1="56.765" y1="46.8694" x2="61.515" y2="42.1194" width="0" layer="19" extent="1-1"/>
+</signal>
 </signals>

Commit message: schematic check-up
initial schematic done, beginning routing
Parts:
- removed 32KHZ: ABS07, ABS07_crys:ABS07
- removed C10, C3, C4: 10uF, microbuilder:0805
- removed C11, C13, C6, C7: 1uF, microbuilder:0805
- removed C12: 2.2uF/16V, microbuilder:0805
- removed C14, C15: 10pF, rcl:C0603
- removed C16: 10uF, rcl:C0603
- removed C17, C18, C19, C20: .1uF, rcl:C0603
- removed C21: 4.7uF, rcl:C0603
- removed CC1: Value, CC3200:RGC0064A
- removed D1, D2, D3: 1N4148, microbuilder:SOD-323
- removed FID1, FID2: FIDUCIAL"", microbuilder:FIDUCIAL_1MM
- removed IC1: (no value), ftdichip-3:QFP48-7X7
- removed J2: (no value), microbuilder:1X05_ROUND_76
- removed Q2, Q3: BSS138, microbuilder:SOT23-WIDE
- removed R14, R4: 10K, microbuilder:0805
- removed R8: 390K, microbuilder:0805
- removed SJ1, SJ2: (no value), microbuilder:SOLDERJUMPER_REFLOW_NOPASTE
- removed SV1: (no value), con-lsta:FE10-2
- removed U$23, U$24, U$25, U$26: MOUNTINGHOLE2.5, microbuilder:MOUNTINGHOLE_2.5_PLATED
- removed U$27: 2.2uH, ABS07_crys:1008INDUCTOR
- removed U$4: Q24FA20H00396, ABS07_crys:Q24FA20H00396
- removed U2: UG-2864HSWEG01, microbuilder:UG-2864HSWEG01_0.96IN_WRAPAROUND
- removed U3: (no value), microbuilder:SOT23-5
- added ANT_PAD: ANT, Antenna:ANT
- added C24: .01uF, rcl:C0603
- added C25, C27: 10uF, rcl:C0603
- added C26: 15pF, rcl:C0603
- added C33: 1pF, rcl:C0402
- added CC3200MOD: CC3200, cc3200mod:CC3200MOD
- added JP3: (no value), pinhead:1X07
- added JP6: (no value), pinhead:2X10/90
- added L1: 3.6nH, Spark:C0402
- added R10, R9: 33, rcl:R0603
- added R16: 2.7K, SparkFun-Resistors:0603-RES
- added R26: 10k, adafruit:R0805
- added R31: 52.3K, resistor:R0805
- added R32: 30.1K, resistor:R0805
- added R33: 0, SparkFun-Resistors:0603-RES
- added R37, R41: 0, adafruit:R0805
- added SOP0, SOP2: (no value), pinhead:1X02
- added U$30: TPS737_DCQ, tps737DCQ:TPS737_DCQ
- added U6: TPS79328DBVRG4, Texas Instruments_By_element14_Batch_1:SOT95P280X145-5N
- added X1, X2: FH12-24S-0.5SH, con-hirose:FH12-24S-0.5SH
- C22: value 4.7uF -> 2.2uF
- C23: value 4.7uF -> .1uF
- JP1: device microbuilder:1X08_ROUND_70 -> SparkFun-Connectors:JST-2-SMD
- R1, R3: device adafruit:R0805 -> rcl:R0603
- R11, R12, R13: device microbuilder:0805 -> rcl:R0603
- R2: value 100k -> 100K; device adafruit:R0805 -> rcl:R0603
- R5: value 10K -> 2.7K; device microbuilder:0805 -> SparkFun-Resistors:0603-RES
- R6, R7: value 10K -> 3.3K; device microbuilder:0805 -> rcl:R0603
- moved C22 217.0 mm to (129.0, 22.0), turned to 270 degrees
- moved C23 215.5 mm to (119.0, 23.0), turned to 270 degrees
- moved R11 170.6 mm to (134.0, 10.0), turned to 90 degrees
- moved R6 169.0 mm to (144.0, 23.0)
- moved R7 161.2 mm to (144.0, 19.0)
- moved R12 137.9 mm to (120.0, 6.00), turned to 90 degrees
- moved R13 134.4 mm to (124.0, 4.00), turned to 90 degrees
- moved R5 118.0 mm to (18.0, 23.0)
- moved FB2 110.6 mm to (90.0, 19.0)
- moved R1 103.3 mm to (94.0, 14.0)
- moved R2 102.0 mm to (99.0, 13.0), turned to 90 degrees
- moved FB1 99.2 mm to (90.0, 23.0)
- moved C1 96.4 mm to (80.0, 19.0), turned to 90 degrees
- moved R3 90.4 mm to (93.0, 11.0), turned to 90 degrees
- moved JP1 90.3 mm to (4.00, 5.00), turned to 90 degrees
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Connections:
- removed net 3.3V: C11.2, C13.2, C4.1, JP1.6, Q2.1, Q3.1, R11.2, R12.2, R5.2, R6.2, R7.2, SJ2.1, U2.6, U2.9, U3.5
- removed net 3V3OUT: IC1.6
- removed net A/R: J2.5, U$1.P$9
- removed net AGND: IC1.45
- removed net AVCC: IC1.46
- removed net CS_3.3V: D1.A, R5.1, U2.13
- removed net CS_5.0V: D1.C, JP1.5
- removed net D0/SCLK/SCK_3.3V: Q3.2, R12.1, U2.18
- removed net D0/SCLK/SCK_5.0V: JP1.2, Q3.3, R14.1
- removed net D1/MOSI/SDA1_3.3V: Q2.2, R11.1, SJ1.1, U2.19
- removed net D1/MOSI/SDA_5.0V: JP1.1, Q2.3, R13.1
- removed net DC/SA0_3.3V: D3.A, R7.1, U2.15
- removed net DC/SA0_5.0V: D3.C, JP1.3
- removed net DCDC_ANA_SW: CC1.38
- removed net DCDC_PA_OUT: CC1.42
- removed net DCDC_PA_SW_N: CC1.41
- removed net DCDC_PA_SW_P: CC1.40
- removed net GAIN: J2.3, U$1.P$10
- removed net LDO_IN1: CC1.36
- removed net LDO_IN2: CC1.25
- removed net N$2: FB1.1, J2.2
- removed net OUTPUT: J2.4, U$1.P$6
- removed net RST_3.3V: D2.A, R6.1, U2.14
- removed net RST_5.0V: D2.C, JP1.4
- removed net VBAT_CC: C19.1, C20.1, C21.1, C22.1, C23.1, CC1.10, CC1.37, CC1.39, CC1.44, CC1.54, IC1.3, IC1.42
- removed net VCCA: U1.1
- removed net VCCB: U1.8
- removed net VCCIOA: IC1.14
- removed net VCCIOB: IC1.31
- removed net VDD: C1.1, FB1.2, U$1.P$2, U$1.P$5
- removed net VDD_ANA1: CC1.48
- removed net VDD_ANA2: CC1.47
- removed net VDD_PA_IN: CC1.33
- removed net VDD_PLL: CC1.24
- removed net VDD_RAM: CC1.49
- removed net VIN: C3.1, JP1.7, R13.2, R14.2, U3.1, U3.3
- removed net XHIGH: CC1.23, U$4.XHIGH
- removed net XLOW: CC1.22, U$4.XLOW
- removed net XTALHIGH: 32KHZ.XLOW, C15.1, CC1.51
- removed net XTALLOW: 32KHZ.XHIGH, C14.2, CC1.52
- new net EN: JP6.17, R26.2, R9.1
- new net GPIO_01/PCK/FLASH_RX: CC3200MOD.P46, JP3.5, JP6.8
- new net GPIO_03/D5: CC3200MOD.P48, JP6.14
- new net GPIO_04/D4: CC3200MOD.P49, JP6.13
- new net GPIO_05/D3: CC3200MOD.P50, JP6.16
- new net GPIO_06/D2: CC3200MOD.P51, JP6.15
- new net GPIO_07/OLED_RST: CC3200MOD.P52
- new net GPIO_09/EN: CC3200MOD.P54, R13.2, U1.3
- new net GPIO_11/MCK: CC3200MOD.P4, R12.2, U1.2
- new net GPIO_12/VS: CC3200MOD.P9, JP6.6
- new net GPIO_13/PHS: CC3200MOD.P10, JP6.5
- new net GPIO_14/D6: CC3200MOD.P5, JP6.11
- new net GPIO_15/D7: CC3200MOD.P6, JP6.12
- new net GPIO_16/D8: CC3200MOD.P7, JP6.9
- new net GPIO_17/D9: CC3200MOD.P8, JP6.10
- new net GSPI_CS: CC3200MOD.P44
- new net GSPI_MISO: CC3200MOD.P42
- new net I2C_SCL: JP6.4, R41.2, R7.1
- new net I2C_SCL/JTAG_TDI: CC3200MOD.P12, JP3.4, R41.1
- new net I2C_SDA: JP6.3, R37.2, R6.1
- new net I2C_SDA/JTAG_TDO: CC3200MOD.P18, JP3.3, R37.1
- new net JTAG_TCK: JP3.2
- new net JTAG_TMS: JP3.1
- new net LDO_2.8V: C22.2, R6.2, R7.2, U1.8
- new net MCK: JP6.7, R10.1
- new net MICA/R: U$1.P$9
- new net MICGAIN: U$1.P$10
- new net MICOUT: U$1.P$6
- new net MICOUT/FLASH_TX: CC3200MOD.P47, JP3.6
- new net MIC_VDD: FB1.1, U$1.P$2, U$1.P$5
- new net N$21: ANT_PAD.FEED2, C33.1, L1.1
- new net N$22: X1.17
- new net N$23: X1.18
- new net N$24: X1.19
- new net N$25: X1.20
- new net N$26: X1.21
- new net N$27: X1.22
- new net N$28: X1.23
- new net N$29: JP6.20
- new net N$30: X1.24
- new net N$31: X1.14
- new net N$32: X1.13
- new net N$33: X1.12
- new net N$34: X1.11
- new net N$35: X2.14
- new net N$36: X1.10
- new net N$37: X1.9
- new net N$38: X1.8
- new net N$39: X1.7
- new net N$40: JP6.19
- new net N$41: X1.6
- new net N$42: X1.5
- new net N$43: X1.4
- new net N$44: X1.3
- new net N$45: X1.2
- new net N$46: X1.1
- new net N$47: CC3200MOD.P45
- new net N$48: X2.13
- new net N$49: C22.1, U6.5
- new net N$50: R11.1, U1.5
- new net N$51: C24.1, U6.4
- new net N$52: X2.12
- new net N$53: R10.2, U1.7
- new net N$54: R9.2, U1.6
- new net N$55: X2.11
- new net N$56: X2.10
- new net N$57: X2.9
- new net N$58: X2.8
- new net N$59: X2.7
- new net N$60: X2.6
- new net N$61: X2.5
- new net N$62: X2.4
- new net N$63: X2.3
- new net N$64: X2.2
- new net N$65: X2.1
- new net N$76: CC3200MOD.P53
- new net N_RESET: CC3200MOD.P35, JP3.7
- new net REGFB: R31.1, R32.2, U$30.NR/FB
- new net REGVOUT: C26.1, R31.2, R33.1, U$30.OUT
- new net SOP0: CC3200MOD.P34, R5.1, SOP0.1
- new net SOP2: CC3200MOD.P23, R16.1, SOP2.1
- new net VBATT: C25.1, JP1.1, U$30.EN, U$30.IN
- new net VCC: C1.1, C23.1, C27.1, CC3200MOD.P36, CC3200MOD.P37, CC3200MOD.P39, CC3200MOD.P40, FB1.2, JP6.2, R11.2, R33.2, SOP0.2, SOP2.2, U1.1, U6.1, U6.3
- net GND: now also ANT_PAD.ANT_GND, ANT_PAD.GND_LEFT, C24.2, C25.2, C26.2, C27.2, C33.2, CC3200MOD.P1, CC3200MOD.P16, CC3200MOD.P2, CC3200MOD.P27, CC3200MOD.P28, CC3200MOD.P30, CC3200MOD.P32, CC3200MOD.P38, CC3200MOD.P43, CC3200MOD.P55, CC3200MOD.P56, CC3200MOD.P57, CC3200MOD.P58, CC3200MOD.P59, CC3200MOD.P60, CC3200MOD.P61, CC3200MOD.P62, CC3200MOD.P63, FB2.1, JP1.2, JP6.1, JP6.18, R12.1, R13.1, R16.2, R26.1, R32.1, R5.2, U$30.GND, U$30.TAB, U1.4, U6.2; no longer C10.1, C11.1, C12.1, C13.1, C14.1, C15.2, C16.2, C17.2, C18.2, C19.2, C20.2, C21.2, C22.2, C3.2, C4.2, CC1.65, IC1.18, IC1.25, IC1.34, IC1.9, JP1.8, R4.1, R8.1, U$4.GND1, U$4.GND2, U2.1, U2.10, U2.12, U2.29, U2.30, U2.8, U3.2
- net N$1: now also X2.15; no longer R4.2, SJ2.2, U2.11
- net N$10: now also R1.2; no longer R1.1
- net N$11: now also R1.1; no longer R1.2
- net N$12: now also X2.19; no longer C6.1, U2.3
- net N$13: now also X2.20; no longer C7.2, U2.4
- net N$14: now also X2.21; no longer C7.1, U2.5
- net N$15: now also X2.22; no longer C10.2, U2.28
- net N$16: now also X2.23; no longer C12.2, U2.27
- net N$17: now also X2.24; no longer SJ1.2, U2.20
- net N$18: now also X1.15; no longer CC1.43, U$27.P2
- net N$19: now also CC3200MOD.P31, L1.2; no longer C16.1, U$27.P1
- net N$20: now also X1.16; no longer C17.1, C18.1, CC1.56, CC1.9
- net N$3: now also X2.16; no longer FB2.1, J2.1
- net N$4: now also X2.17; no longer R8.2, U2.26
- net N$6: now also X2.18; no longer C6.2, U2.2
Other:
- board size 160 x 100 mm -> 160 x 30 mm

Commit message: initial board push
first revision of board is...done! This revision still needs to:
-review antenna trace with expert
-clean up some of the routing
-be reviewed by non-john member of the team
Parts:
- removed C1, C5: 2.2uF, adafruit:C0805K
- removed C2, C9: 0.1uF, adafruit:C0805K
- removed C8: 0.47uF, adafruit:C0805K
- removed FB1, FB2: FERRITE, microbuilder:0805
- removed JP6: (no value), pinhead:2X10/90
- removed Q1: CMA-4544PF-W, adafruit:9.7ELECTRET
- removed R2: 100K, rcl:R0603
- removed R26: 10k, adafruit:R0805
- removed R3: 2.2K, rcl:R0603
- removed R33: 0, SparkFun-Resistors:0603-RES
- removed R37, R41: 0, adafruit:R0805
- removed U$1: MAX9814TDFN14, adafruit:TDFN14_3X3MM
- removed X1, X2: FH12-24S-0.5SH, con-hirose:FH12-24S-0.5SH
- added R4: 100k, SparkFun-Resistors:0603-RES
- added SV1: (no value), con-dil:16P
- R1: value 150k -> 10k; device rcl:R0603 -> resistor:R0603
- moved R11 82.1 mm to (52.5, 20.0)
- moved R7 81.2 mm to (63.0, 24.1), turned to 270 degrees
- moved R6 80.0 mm to (64.0, 20.8), turned to 180 degrees
- moved R9 73.9 mm to (61.0, 17.5), turned to 180 degrees
- moved U1 72.9 mm to (57.0, 19.5)
- moved R10 72.8 mm to (63.5, 19.0), turned to 180 degrees
- moved C22 69.9 mm to (59.1, 24.8), turned to 90 degrees
- moved R13 69.7 mm to (54.3, 5.99), turned to 180 degrees
- moved C24 69.7 mm to (59.6, 22.3), turned to 0 degrees
- moved R12 68.6 mm to (51.5, 8.12)
- moved U6 68.0 mm to (56.0, 23.0)
- moved C23 64.1 mm to (55.0, 26.0), turned to 45 degrees
- moved C27 45.7 mm to (16.0, 3.00), turned to 180 degrees
- moved R1 30.2 mm to (63.9, 16.3), turned to 90 degrees
- moved R16 26.5 mm to (35.2, 28.2)
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Connections:
- net N$19 renamed MCU_RF
- removed net I2C_SCL: JP6.4, R41.2, R7.1
- removed net I2C_SDA: JP6.3, R37.2, R6.1
- removed net INPUT: C9.2, Q1.+, R3.1
- removed net MICA/R: U$1.P$9
- removed net MICGAIN: U$1.P$10
- removed net MICOUT: U$1.P$6
- removed net MIC_VDD: FB1.1, U$1.P$2, U$1.P$5
- removed net N$1: X2.15
- removed net N$10: R1.2, R2.2, U$1.P$14
- removed net N$11: R1.1, R3.2, U$1.P$13
- removed net N$12: X2.19
- removed net N$13: X2.20
- removed net N$14: X2.21
- removed net N$15: X2.22
- removed net N$16: X2.23
- removed net N$17: X2.24
- removed net N$18: X1.15
- removed net N$20: X1.16
- removed net N$22: X1.17
- removed net N$23: X1.18
- removed net N$24: X1.19
- removed net N$25: X1.20
- removed net N$26: X1.21
- removed net N$27: X1.22
- removed net N$28: X1.23
- removed net N$29: JP6.20
- removed net N$3: X2.16
- removed net N$30: X1.24
- removed net N$31: X1.14
- removed net N$32: X1.13
- removed net N$33: X1.12
- removed net N$34: X1.11
- removed net N$35: X2.14
- removed net N$36: X1.10
- removed net N$37: X1.9
- removed net N$38: X1.8
- removed net N$39: X1.7
- removed net N$4: X2.17
- removed net N$40: JP6.19
- removed net N$41: X1.6
- removed net N$42: X1.5
- removed net N$43: X1.4
- removed net N$44: X1.3
- removed net N$45: X1.2
- removed net N$46: X1.1
- removed net N$48: X2.13
- removed net N$49: C22.1, U6.5
- removed net N$5: C9.1, U$1.P$8
- removed net N$52: X2.12
- removed net N$55: X2.11
- removed net N$56: X2.10
- removed net N$57: X2.9
- removed net N$58: X2.8
- removed net N$59: X2.7
- removed net N$6: X2.18
- removed net N$60: X2.6
- removed net N$61: X2.5
- removed net N$62: X2.4
- removed net N$63: X2.3
- removed net N$64: X2.2
- removed net N$65: X2.1
- removed net N$7: C8.1, U$1.P$12
- removed net N$8: C2.1, U$1.P$1
- removed net N$9: C5.1, U$1.P$3
- removed net REGVOUT: C26.1, R31.2, R33.1, U$30.OUT
- net EN: now also R1.2, SV1.11; no longer JP6.17, R26.2
- net GND: now also C22.2, JP1.1, R1.1, R4.2; no longer C1.2, C2.2, C26.2, C5.2, C8.2, FB2.1, FB2.2, JP1.2, JP6.1, JP6.18, Q1.-, R2.1, R26.1, U$1.P$11, U$1.P$4, U$1.P$7, U$1.P$THERMAL
- net GPIO_01/PCK/FLASH_RX: now also SV1.2; no longer JP3.5, JP6.8
- net GPIO_03/D5: now also SV1.3; no longer JP6.14
- net GPIO_04/D4: now also SV1.6; no longer JP6.13
- net GPIO_05/D3: now also SV1.5; no longer JP6.16
- net GPIO_06/D2: now also SV1.4; no longer JP6.15
- net GPIO_12/VS: now also SV1.14; no longer JP6.6
- net GPIO_13/PHS: now also SV1.13; no longer JP6.5
- net GPIO_14/D6: now also SV1.8; no longer JP6.11
- net GPIO_15/D7: now also SV1.7; no longer JP6.12
- net GPIO_16/D8: now also SV1.10; no longer JP6.9
- net GPIO_17/D9: now also SV1.9; no longer JP6.10
- net I2C_SCL/JTAG_TDI: now also R7.1, SV1.15; no longer R41.1
- net I2C_SDA/JTAG_TDO: now also R6.1, SV1.16; no longer R37.1
- net JTAG_TCK: now also CC3200MOD.P21
- net JTAG_TMS: now also CC3200MOD.P22, R4.1
- net LDO_2.8V: now also C22.1, U6.5; no longer C22.2
- net MCK: now also SV1.12; no longer JP6.7
- net MICOUT/FLASH_TX: now also JP3.5, SV1.1; no longer JP3.6
- net REGFB: now also C26.2
- net VBATT: now also JP1.2; no longer JP1.1
- net VCC: now also C26.1, R31.2, U$30.OUT; no longer C1.1, FB1.2, JP6.2, R33.2
Routing:
- net GPIO_01/PCK/FLASH_RX: track 0.00 -> 97.8 mm, vias 0 -> 1
- net I2C_SDA/JTAG_TDO: track 0.00 -> 90.9 mm, vias 0 -> 3
- net MICOUT/FLASH_TX: track 0.00 -> 87.1 mm
- net I2C_SCL/JTAG_TDI: track 0.00 -> 80.7 mm, vias 0 -> 4
- net SOP2: track 0.00 -> 53.2 mm, vias 0 -> 1
- net JTAG_TMS: track 0.00 -> 50.2 mm, vias 0 -> 1
- net JTAG_TCK: track 0.00 -> 45.2 mm, vias 0 -> 2
- net GPIO_04/D4: track 0.00 -> 41.4 mm
- net GPIO_06/D2: track 0.00 -> 35.9 mm, vias 0 -> 1
- net N_RESET: track 0.00 -> 35.9 mm
- net GPIO_03/D5: track 0.00 -> 34.9 mm
- net GPIO_05/D3: track 0.00 -> 31.6 mm
- net GPIO_12/VS: track 0.00 -> 30.4 mm, vias 0 -> 1
- net GPIO_16/D8: track 0.00 -> 28.3 mm
- net GPIO_14/D6: track 0.00 -> 28.1 mm
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- added copper zone on layer 1, net GND
- added copper zone on layer 2, net GND
- added copper zone on layer 1, net N$1
- added copper zone on layer 1, net N$12
- added copper zone on layer 1, net N$2
- added copper zone on layer 1, net N$3
- added copper zone on layer 1, net N$4
- added copper zone on layer 1, net N$57
- added copper zone on layer 1, net N$6
- added copper zone on layer 16, net N$71
- added copper zone on layer 1, net VCC
- added copper zone on layer 15, net VCC
Other:
- board size 160 x 30 mm -> 78 x 30.5 mm
- board text added: "TODO: figure out where to put the connector..."
